Commit message: 增加相机点云发布和激光雷达

File: urdf/hhfc/urdf/hhfc.urdf (robot description, URDF)
Before this commit: robot hhfc, 16 links, 15 joints
Links:
- added link lidar_link, mass 0.2; collision cylinder length=0.05 radius=0.03; visual cylinder length=0.05 radius=0.03
Joints:
- added joint lidar_joint: type fixed, parent base_thorax, child lidar_link, origin xyz=0.1 0 0.5 rpy=0 0 0

Commit message: update

File: urdf/hhfc/urdf/hhfc.urdf (robot description, URDF)
Before this commit: robot hhfc, 17 links, 16 joints
Links:
- link lidar_link: mass 0.2 -> 0.02
