Commit message: update

File: urdf/efc/urdf/efc_23dof_fake_lim.urdf (robot description, URDF)
Before this commit: robot sr02h_v1, 26 links, 25 joints
Links:
- removed link camera_link
- link base_link: geometry visual mesh filename=../meshes/base_link.STL
- link head_link: geometry visual mesh filename=../meshes/head.STL
- link left_ankle_pitch_link: geometry visual mesh filename=../meshes/left_ankle_pitch.STL
- link left_ankle_roll_link: geometry collision cylinder length=0.16 radius=0.01; collision cylinder length=0.16 radius=0.01
- link left_elbow_pitch_link: geometry collision cylinder length=0.3 radius=0.04; visual mesh filename=../meshes/left_elbow_pitch.STL
- link left_elbow_yaw_link: geometry visual mesh filename=../meshes/left_elbow_yaw.STL
- link left_hip_pitch_link: geometry visual mesh filename=../meshes/left_hip_pitch.STL
- link left_hip_roll_link: geometry collision cylinder length=0.1 radius=0.055; visual mesh filename=../meshes/left_hip_roll.STL
- link left_hip_yaw_link: geometry collision cylinder length=0.2 radius=0.052; visual mesh filename=../meshes/left_hip_yaw.STL
- link left_knee_link: geometry collision cylinder length=0.26 radius=0.052; visual mesh filename=../meshes/left_knee.STL
- link left_shoulder_pitch_link: geometry visual mesh filename=../meshes/left_shoulder_pitch.STL
- link left_shoulder_roll_link: geometry visual mesh filename=../meshes/left_shoulder_roll.STL
- link left_shoulder_yaw_link: geometry collision cylinder length=0.2 radius=0.04; visual mesh filename=../meshes/left_shoulder_yaw.STL
- link right_ankle_pitch_link: geometry visual mesh filename=../meshes/right_ankle_pitch.STL
- link right_ankle_roll_link: geometry collision cylinder length=0.16 radius=0.01; collision cylinder length=0.16 radius=0.01
- link right_elbow_pitch_link: geometry collision cylinder length=0.3 radius=0.04; visual mesh filename=../meshes/right_elbow_pitch.STL
- link right_elbow_yaw_link: geometry visual mesh filename=../meshes/right_elbow_yaw.STL
- link right_hip_pitch_link: geometry visual mesh filename=../meshes/right_hip_pitch.STL
- link right_hip_roll_link: geometry collision cylinder length=0.1 radius=0.055; visual mesh filename=../meshes/right_hip_roll.STL
- link right_hip_yaw_link: geometry collision cylinder length=0.2 radius=0.052; visual mesh filename=../meshes/right_hip_yaw.STL
- link right_knee_link: geometry collision cylinder length=0.26 radius=0.052; visual mesh filename=../meshes/right_knee.STL
- link right_shoulder_pitch_link: geometry visual mesh filename=../meshes/right_shoulder_pitch.STL
- link right_shoulder_roll_link: geometry visual mesh filename=../meshes/right_shoulder_roll.STL
- link right_shoulder_yaw_link: geometry collision cylinder length=0.2 radius=0.04; visual mesh filename=../meshes/right_shoulder_yaw.STL
- link waist_link: geometry collision box size=0.2 0.26 0.5; visual mesh filename=../meshes/upper_body.STL
Joints:
- removed joint camera_joint
- joint head_joint: type revolute -> fixed
