Commit message: update

File: urdf/efc/urdf/efc.urdf (robot description, URDF)
Before this commit: robot sr02h_v1, 26 links, 25 joints
Joints:
- joint camera_joint: origin xyz=0.1 0.0 0.0 rpy=-2.181661564992912 0.0 -1.57079632679489661923 -> xyz=0.0907988662332928 0.01 0.0 rpy=-2.181661564992912 0.0 -1.57079632679489661923

Commit message: hike in the world demo

File: urdf/efc/urdf/efc.urdf (robot description, URDF)
Before this commit: robot sr02h_v1, 26 links, 25 joints
Joints:
- joint camera_joint: origin xyz=0.0907988662332928 0.01 0.0 rpy=-2.181661564992912 0.0 -1.57079632679489661923 -> xyz=0.0907988662332928 0.01 0.0 rpy=-0.00530447 0.83774397 0.01191416

Commit message: parkour policy

File: urdf/efc/urdf/efc.urdf (robot description, URDF)
Before this commit: robot sr02h_v1, 26 links, 25 joints
Links:
- link camera_link: geometry visual box size=0.02 0.1 0.02

Commit message: update

File: urdf/efc/urdf/efc.urdf (robot description, URDF)
Before this commit: robot sr02h_v1, 26 links, 25 joints
Joints:
- joint camera_joint: origin xyz=0.0907988662332928 0.01 0.0 rpy=-0.00530447 0.83774397 0.01191416 -> xyz=0.081 -0.047 0.019 rpy=0.0 0.6108652382 0.0

Commit message: update

File: urdf/efc/urdf/efc.urdf (robot description, URDF)
Before this commit: robot sr02h_v1, 26 links, 25 joints
Joints:
- joint camera_joint: origin xyz=0.081 -0.047 0.019 rpy=0.0 0.6108652382 0.0 -> xyz=0.12623021 0.0475 0.22489942 rpy=0.0 0.8726646259971648 0.0
