Commit message: camera processing update

File: urdf/efc/urdf/efc.urdf (robot description, URDF)
Before this commit: robot sr02h_v1, 26 links, 25 joints
Links:
- link left_hip_yaw_link: geometry collision cylinder length=0.2 radius=0.062; visual mesh filename=package://bitbot_gz/urdf/efc/meshes/left_hip_yaw.STL
- link left_knee_link: geometry collision cylinder length=0.26 radius=0.055; visual mesh filename=package://bitbot_gz/urdf/efc/meshes/left_knee.STL
- link right_knee_link: geometry collision cylinder length=0.26 radius=0.055; visual mesh filename=package://bitbot_gz/urdf/efc/meshes/right_knee.STL
Joints:
- joint camera_joint: origin xyz=0.12623021 0.0475 0.22489942 rpy=0.0 0.8726646259971648 0.0 -> xyz=0.12380269 -0.0475 0.22030226 rpy=0.0 0.8726646259971648 0.0
